Commit message: adding a camera depth frame

File: nao_description/urdf/naoV40_generated_urdf/nao.urdf (robot description, URDF)
Before this commit: robot NaoH25V40, 83 links, 82 joints
Links:
- added link CameraDepth_frame
Joints:
- added joint CameraDepth_joint: type fixed, parent Head, child CameraDepth_frame, origin xyz=0.02 -0.04708 0.13 rpy=-2.0043951 0 -1.5708

File: nao_description/urdf/naoV40_generated_urdf/nao_sensors.xacro (robot description, xacro)
@@ -342,3 +342,9 @@
 		<axis xyz="0 0 0"/>
 	</joint>
+	<link name="CameraDepth_frame"/>
+        <joint name="CameraDepth_joint" type="fixed">
+	        <parent link="Head"/>
+	        <child link="CameraDepth_frame"/>
+	        <origin rpy="-2.0043951 0 -1.5708" xyz="0.02 -0.04708 0.13"/>
+        </joint>
 </robot>
